Commit message: Scale down collision meshes to prevent false collisions
Add scale="0.95 0.95 0.95" to all collision geometry meshes.
SolidWorks-exported URDFs use full-detail STL files for collision
detection, which causes frequent false-positive collisions when
joints rotate. Scaling down by 5% provides clearance while
maintaining meaningful collision detection.

File: moveit_ws/src/my_robot_description/urdf/my_robot_description.urdf (robot description, URDF)
Before this commit: robot my_robot_description, 6 links, 5 joints
Links:
- link Link_4: geometry collision mesh filename=package://my_robot_description/meshes/Link_4.STL scale=0.95 0.95 0.95; visual mesh filename=package://my_robot_description/meshes/Link_4.STL
- link base_link: geometry collision mesh filename=package://my_robot_description/meshes/base_link.STL scale=0.95 0.95 0.95; visual mesh filename=package://my_robot_description/meshes/base_link.STL
- link grab: geometry collision mesh filename=package://my_robot_description/meshes/grab.STL scale=0.95 0.95 0.95; visual mesh filename=package://my_robot_description/meshes/grab.STL
- link link_1: geometry collision mesh filename=package://my_robot_description/meshes/link_1.STL scale=0.95 0.95 0.95; visual mesh filename=package://my_robot_description/meshes/link_1.STL
- link link_2: geometry collision mesh filename=package://my_robot_description/meshes/link_2.STL scale=0.95 0.95 0.95; visual mesh filename=package://my_robot_description/meshes/link_2.STL
- link link_3: geometry collision mesh filename=package://my_robot_description/meshes/link_3.STL scale=0.95 0.95 0.95; visual mesh filename=package://my_robot_description/meshes/link_3.STL
